File: effectiveRangeRelay.kicad_pcb (KiCad board)
At the start: 4 copper layers, 27.6 x 41.4 mm, 24 parts, among them J1 RELAY_CTRL, J2 OUT, J3 RELAY_PWR, K1 J107F1CS125VDC.36, Q1 2N7002, U1 APC-817C1-SL

Commit message: Bumping release from 2.1.0 to 2.2.0
Other:
- board text added: "RelayDevice v2.2.0"
- board text removed: "RelayDevice v2.1.0"
Changed lines of the file:
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@@
 	(title_block
 		(title "Effective Range RelayDevice")
-		(date "2024-04-16")
+		(date "2024-06-17")
 		(rev "v2.1.0")
 		(company "Effective Range Kft.")
@@
 		(layer "Edge.Cuts")
 	)
-	(gr_text "RelayDevice v2.1.0"
+	(gr_text "RelayDevice v2.2.0"
 		(at 129.921 105.029 90)
 		(layer "F.Cu")
